File: hardware/Badge-HackGDL-2026.kicad_pcb (KiCad board)
At the start: 2 copper layers, 143 parts, among them J1 Conn_01x20, J10 Battery, J2 Conn_01x04_Pin, J9 Add_On, P4 USB_C_Plug_USB2.0, Q1 DMG3415U-7, SW1 ON, SW2 SW_Push, SW3 SW_Push, U2 TP4056, U4 MT3608, U5 AP2114H-3.3, U6 W25N02KVZEIR, U7 EA3059, Y1 Crystal, Y2 24MHz

Commit message: feat(Hw):Update_Schematic_And_Floorplan
Parts:
- added FID1: Camera, Footprints:Camera, F.Cu at (136.3, 49.0)
- C10, C11, C12, C13, C14, C15, C16, C17, C58, C59, C61, C7, C8, C86, C9, D3, D4, D5, D6, L4, L5, L6, L7, R1, R12, R20, R21, R22, R23, R24, R38, R39, R41, R42, R43, R5, R6, R7, R8, U7: moved to B.Cu
- moved J2 212.7 mm to (278.9, 87.8)
- moved C5 212.2 mm to (246.6, 125.2)
- moved SW2 211.4 mm to (253.2, 116.7)
- moved SW3 211.4 mm to (253.2, 123.8)
- moved R9 209.0 mm to (258.6, 119.6), turned to 180 degrees
- moved C4 200.4 mm to (240.0, 98.5), turned to 90 degrees
- moved C60 198.9 mm to (259.3, 117.2)
- moved C3 197.5 mm to (237.3, 95.1)
- moved R25 195.8 mm to (246.6, 126.1)
- moved Y2 194.4 mm to (237.7, 97.8), turned to 90 degrees
- moved R26 194.3 mm to (246.6, 123.7)
- moved C27 190.2 mm to (233.2, 98.7)
- moved C26 189.6 mm to (233.2, 92.8)
- moved C30 187.9 mm to (233.2, 96.5)
- moved C23 186.5 mm to (227.4, 101.3), turned to -90 degrees
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Routing:
- net GND: track 0.00 -> 15.9 mm, vias 0 -> 1
- net VCC: track 0.00 -> 12.7 mm, vias 0 -> 2
- net /Buck_Converter/EN3: track 0.00 -> 4.19 mm
- net /Buck_Converter/EN4: track 0.00 -> 4.18 mm
- net /Buck_Converter/EN1: track 0.00 -> 4.08 mm
- net /Buck_Converter/EN2: track 0.00 -> 4.01 mm
- added copper zone on B.Cu, net +1V8
- added copper zone on B.Cu, net +3V3
- added copper zone on B.Cu, net /Buck_Converter/FB1
- added copper zone on B.Cu, net /Buck_Converter/FB2
- added copper zone on B.Cu, net /Buck_Converter/FB3
- added copper zone on B.Cu, net /Buck_Converter/FB4
- added copper zone on B.Cu, net /Buck_Converter/LX1
- added copper zone on B.Cu, net /Buck_Converter/LX2
- added copper zone on B.Cu, net /Buck_Converter/LX3
- added copper zone on B.Cu, net /Buck_Converter/LX4
- added copper zone on B.Cu, net /Buck_Converter/VCC_DDR
- added copper zone on B.Cu, net /Buck_Converter/v_0.9v
- added copper zone on B.Cu, net VCC
Other:
- board outline added: 23 x 15.5 mm

Commit message: feat(Hw):Update_Schematic
Parts:
- removed D3, D4, D5, D6: LED, LED_SMD:LED_0603_1608Metric
- removed R10, R28, R30: 0R, Resistor_SMD:R_0402_1005Metric
- removed R39: 330, Resistor_SMD:R_0402_1005Metric
- removed R41, R42, R43: 50, Resistor_SMD:R_0603_1608Metric
- R44: value 10.7K -> 12.3K
- R45: value 10K -> 9.09K
- moved C70 172.9 mm to (197.0, 42.1), turned to 180 degrees
- moved R32 168.9 mm to (196.9, 44.6)
- moved C54 167.5 mm to (207.1, 95.8), turned to 90 degrees
- moved C71 165.3 mm to (189.3, 40.3)
- moved J10 160.6 mm to (227.2, 26.7)
- moved R19 155.2 mm to (206.2, 95.8), turned to 90 degrees
- moved R13 154.9 mm to (205.2, 95.8), turned to 90 degrees
- moved R31 154.6 mm to (182.7, 44.1), turned to -90 degrees
- moved R11 151.3 mm to (171.5, 20.2)
- moved R45 133.1 mm to (190.6, 39.1)
- moved R44 131.1 mm to (188.7, 39.1)
- moved SW1 130.1 mm to (162.4, 25.6), turned to -90 degrees
- moved R46 127.6 mm to (185.5, 46.0)
- moved C18 123.3 mm to (166.0, 28.0), turned to -90 degrees
- moved U2 109.3 mm to (191.0, 44.0), turned to 180 degrees
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Connections:
- C11 pad 1: /Buck_Converter/v_0.9v -> /MCU/VDD_ARM
- C12 pad 1: /Buck_Converter/v_0.9v -> /MCU/VDD_ARM
- C19 pad 2: /Otros/LEFT -> /MCU/LEFT
- C2 pad 2: /Otros/UP -> /MCU/UP
- C23 pad 1: /Buck_Converter/v_0.9v -> /MCU/VDD_ARM
- C24 pad 1: /Buck_Converter/v_0.9v -> /MCU/VDD_ARM
- C25 pad 1: /Buck_Converter/v_0.9v -> /MCU/VDD_ARM
- C26 pad 1: /Buck_Converter/v_0.9v -> /MCU/VDD_ARM
- C27 pad 1: /Buck_Converter/v_0.9v -> /MCU/VDD_ARM
- C33 pad 2: /Otros/RIGHT -> /MCU/RIGHT
- C37 pad 2: /Otros/DOWN -> /MCU/DOWN
- C43 pad 2: /Otros/PICTURE -> /MCU/PICTURE
- L6 pad 2: /Buck_Converter/v_0.9v -> /MCU/VDD_ARM
- R6 pad 1: /Buck_Converter/v_0.9v -> /MCU/VDD_ARM
- SW4 pad 2: /Otros/UP -> /MCU/UP
- SW5 pad 2: /Otros/LEFT -> /MCU/LEFT
- SW6 pad 2: /Otros/RIGHT -> /MCU/RIGHT
- SW7 pad 2: /Otros/DOWN -> /MCU/DOWN
- SW8 pad 2: /Otros/PICTURE -> /MCU/PICTURE
- U8 pad 10: /Buck_Converter/v_0.9v -> /MCU/VDD_ARM
- U8 pad 103: /Buck_Converter/v_0.9v -> /MCU/VDD_ARM
- U8 pad 116: /Buck_Converter/v_0.9v -> /MCU/VDD_ARM
- U8 pad 12: /MCU/PB2 -> /MCU/PICTURE
- U8 pad 14: unconnected-(U8A-SDMMC0_D0/UART2_RX_M0/PWM8_M0/GPIO3_A3_U-Pad14) -> /MCU/LEFT
- U8 pad 15: unconnected-(U8A-SDMMC0_CLK/UART5_RTS_M0/I2C0_SCL_M2/JTAG_LPMCU_TC_K_M1/PWM10_M0/GPIO3_A4_D-Pad15) -> /MCU/RIGHT
- U8 pad 16: unconnected-(U8A-SDMMC0_CMD/UART5_CTS_M0/I2C0_SDA_M2/JTAG_LPMCU_T_MS_M1/PWM11_IR_M0/GPIO3_A5_U-Pad16) -> /MCU/DOWN
- U8 pad 17: unconnected-(U8A-SDMMC0_D3/UART5_TX_M0/JTAG_CPU_TMS_M0/JTAG_HPMCU__TMS_M1/GPIO3_A6_U-Pad17) -> /MCU/UP
- U8 pad 23: Net-(U8A-SARADC_IN0/GPI4_C0_Z) -> /MCU/RECOVERY
- U8 pad 24: Net-(U8A-SARADC_USB_AVDD1V8) -> +1V8
- U8 pad 51: /Buck_Converter/v_0.9v -> /MCU/VDD_ARM
- U8 pad 54: /Buck_Converter/v_0.9v -> /MCU/VDD_ARM
- U8 pad 55: /Buck_Converter/v_0.9v -> /MCU/VDD_ARM
- U8 pad 67: /Buck_Converter/v_0.9v -> /MCU/VDD_ARM
- U8 pad 71: /Buck_Converter/v_0.9v -> /MCU/VDD_ARM
- U8 pad 78: /MCU/PB1 -> unconnected-(U8C-UART4_TX_M0/PWM7_IR_M1/SPI1_CS1_M0/VI_CIF_D1__M1/GPIO1_B1_D-Pad78)
- U8 pad 82: /Buck_Converter/v_0.9v -> /MCU/VDD_ARM
- U8 pad 93: /MCU/DIN_IR -> unconnected-(U8C-VO_LCDC_D5/VI_CIF_D4_M1/PWM5_M2/I2C4_SCL_M1/_SDMMC1_CLK_M1/SPI0_MOSI_M0/GPIO1_C2_D-Pad93)
Routing:
- added copper zone on B.Cu, net /MCU/VDD_ARM
- removed copper zone on B.Cu, net /Buck_Converter/v_0.9v

Commit message: feat(Hw):Update_Schematic_And_Floorplan
Parts:
- removed C21, C22: 22uF, Capacitor_SMD:C_0402_1005Metric
- removed D9: SS34, Diode_SMD:D_SMA
- removed L1: 4.7uH, Footprints:LQH5BPN
- removed R37: 110K, Resistor_SMD:R_0603_1608Metric
- removed R40: 15K, Resistor_SMD:R_0603_1608Metric
- removed U4: MT3608, Package_TO_SOT_SMD:SOT-23-6
- added R10: 4.7K, Capacitor_SMD:C_0603_1608Metric, F.Cu at (82.5, 61.1)
- added R4: 4.7K, Capacitor_SMD:C_0603_1608Metric, F.Cu at (82.5, 58.6)
- C1, C18, C19, C2, C20, C23, C24, C25, C26, C27, C28, C29, C3, C30, C31, C32, C33, C34, C35, C36, C37, C38, C39, C4, C40, C41, C42, C43, C48, C49, C51, C52, C54, C6, C62, C63, C64, C65, C70, C71, D1, D12, D16, D8, F1, FB1, FB2, J1, J10, P4, Q1, R11, R13, R14, R15, R16, R17, R18, R19, R2, R27, R29, R3, R31, R32, R33, R34, R35, R36, R44, R45, R46, SW1, U2, U5, U6, U8, Y1, Y2: moved to B.Cu
- FID1: footprint Footprints:Camera -> Footprints:Untitled
- SW8: footprint Button_Switch_SMD:SW_SPST_TL3342 -> Footprints:Button_6.6x6.5; moved to B.Cu
- moved C19 197.6 mm to (231.2, 74.1), turned to 180 degrees
- moved C2 197.6 mm to (231.2, 71.6), turned to 180 degrees
- moved C33 197.6 mm to (231.2, 76.6), turned to 180 degrees
- moved C37 197.6 mm to (231.2, 79.1), turned to 180 degrees
- moved C43 197.6 mm to (231.2, 81.6), turned to 180 degrees
- moved SW5 184.6 mm to (211.3, 82.4)
- moved SW7 184.4 mm to (211.3, 92.2)
- moved SW6 184.3 mm to (211.3, 72.6)
- moved SW4 184.3 mm to (211.3, 62.9)
- moved R36 139.8 mm to (95.4, 111.8), turned to 90 degrees
- moved U6 134.6 mm to (94.8, 117.8), turned to -90 degrees
- moved C4 134.3 mm to (105.8, 99.1), turned to 0 degrees
- moved C51 131.8 mm to (92.4, 123.3), turned to 180 degrees
- moved Y2 131.4 mm to (106.4, 101.4), turned to 0 degrees
- moved C52 131.0 mm to (92.4, 124.2), turned to 180 degrees
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Connections:
- P4 pad A6: /USB/2_DP -> /MCU/D+
- P4 pad A7: /USB/2_DN -> /MCU/D-
- SW1 pad 1: Net-(D12-K) -> VCC
- SW1 pad 2: VCC -> Net-(D12-K)
Other:
- board size 23 x 15.5 mm -> 150 x 100 mm

Commit message: feat(Hw):Update_Floorplan_And_Route
Parts:
- added C21: 100nF, Capacitor_SMD:C_0402_1005Metric, F.Cu at (198.7, 49.3)
- added D7: WS2812E-1313, Footprints:WS2812E-1313, F.Cu at (198.7, 48.0)
- added R28: 470R, Resistor_SMD:R_0603_1608Metric, F.Cu at (196.8, 48.0)
- C5, C60, R10, R25, R26, R4, R9, SW2, SW3: moved to B.Cu
- J2: footprint Connector_PinHeader_2.54mm:PinHeader_1x04_P2.54mm_Vertical -> Footprints:4 Pin 2.54mm; moved to B.Cu
- moved J2 202.7 mm to (76.4, 79.7), turned to 180 degrees
- moved R9 160.4 mm to (101.0, 90.0)
- moved SW2 160.3 mm to (95.5, 88.1), turned to 180 degrees
- moved C60 160.2 mm to (101.6, 88.8)
- moved SW3 136.7 mm to (116.6, 120.8), turned to 180 degrees
- moved R26 135.3 mm to (111.3, 122.7)
- moved R25 135.3 mm to (111.3, 121.8), turned to 180 degrees
- moved C5 135.2 mm to (111.4, 123.7), turned to 180 degrees
- moved C43 126.6 mm to (112.8, 36.8), turned to -90 degrees
- moved R13 42.0 mm to (107.4, 116.1), turned to 180 degrees
- moved R19 40.2 mm to (107.4, 117.1), turned to 180 degrees
- moved C54 38.5 mm to (107.4, 118.0), turned to 180 degrees
- moved U5 21.2 mm to (110.9, 55.1)
- moved C31 21.2 mm to (106.9, 58.6)
- moved C32 19.9 mm to (106.9, 52.4), turned to -90 degrees
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Connections:
- U8 pad 104: unconnected-(U8D-UART0_TX_M1/I2C1_SDA_M1/VO_LCDC_D17/PWM6_M1_/GPIO2_B1_D_1-Pad104) -> /MCU/UP
- U8 pad 105: unconnected-(U8D-UART0_TX_M1/I2C1_SDA_M1/VO_LCDC_D17/PWM6_M1_/GPIO2_B1_D_2-Pad105) -> /MCU/RIGHT
- U8 pad 106: unconnected-(U8D-UART0_CTS_M1/I2S0_SDO1_SDI3/VO_LCDC_D15/PWM_4_M1/I2C3_SDA_M0/PRELIGHT_TRIG_OUT/GPIO2_A7_D-Pad106) -> /MCU/LEFT
- U8 pad 107: unconnected-(U8D-UART0_RTS_M1/I2S0_SDO2_SDI2/VO_LCDC_D14/PWM_2_M1/I2C3_SCL_M0/FLASH_TRIG_OUT/GPIO2_A6_D-Pad107) -> /MCU/DOWN
- U8 pad 12: /MCU/PICTURE -> unconnected-(U8A-SDMMC0_D1/UART2_TX_M0/PWM9_M0/GPIO3_A2_U-Pad12)
- U8 pad 14: /MCU/LEFT -> unconnected-(U8A-SDMMC0_D0/UART2_RX_M0/PWM8_M0/GPIO3_A3_U-Pad14)
- U8 pad 15: /MCU/RIGHT -> unconnected-(U8A-SDMMC0_CLK/UART5_RTS_M0/I2C0_SCL_M2/JTAG_LPMCU_TC_K_M1/PWM10_M0/GPIO3_A4_D-Pad15)
- U8 pad 16: /MCU/DOWN -> unconnected-(U8A-SDMMC0_CMD/UART5_CTS_M0/I2C0_SDA_M2/JTAG_LPMCU_T_MS_M1/PWM11_IR_M0/GPIO3_A5_U-Pad16)
- U8 pad 17: /MCU/UP -> unconnected-(U8A-SDMMC0_D3/UART5_TX_M0/JTAG_CPU_TMS_M0/JTAG_HPMCU__TMS_M1/GPIO3_A6_U-Pad17)
- U8 pad 85: unconnected-(U8C-VO_LCDC_CLK/VI_CIF_CLKO_M1/I2C3_SCL_M1/UART5__TX_M1/PWM11_IR_M2/AUD_DSM_N/GPIO1_D3_D-Pad85) -> /MCU/PICTURE
- U8 pad 93: unconnected-(U8C-VO_LCDC_D5/VI_CIF_D4_M1/PWM5_M2/I2C4_SCL_M1/_SDMMC1_CLK_M1/SPI0_MOSI_M0/GPIO1_C2_D-Pad93) -> /MCU/DIN_IR
Routing:
- net /Cam/CSI_SDA: track 0.00 -> 47.6 mm
- net /MCU/DEBUG_RX: track 0.00 -> 46.4 mm
- net /Cam/CSI_SCK: track 0.00 -> 45.2 mm
- net /Cam/MCSI_RST: track 0.00 -> 43.9 mm, vias 0 -> 2
- net /MCU/DEBUG_TX: track 0.00 -> 43.7 mm
- net VBUS: track 0.00 -> 37.9 mm
- net /Cam/MCSI_MCLK: track 0.00 -> 37.1 mm
- net /Cam/MCSI_D1N: track 0.00 -> 36.9 mm
- net /Cam/MCSI_D1P: track 0.00 -> 36.3 mm
- net /Cam/MCSI_CKN: track 0.00 -> 35.0 mm
- net /Cam/MCSI_CKP: track 0.00 -> 34.4 mm
- net /MCU/D-: track 0.00 -> 34.2 mm
- net /MCU/D+: track 0.00 -> 33.6 mm
- net /Cam/MCSI_D0N: track 0.00 -> 32.6 mm
- net /Cam/MCSI_D0P: track 0.00 -> 32.0 mm
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- added copper zone on B.Cu, net +BATT

Commit message: feat(Hw):Update_Route
Parts:
- moved C31 14.2 mm to (92.6, 58.4)
- moved U5 14.2 mm to (96.7, 54.9)
- moved C32 7.83 mm to (99.4, 50.0), turned to 0 degrees
- moved C10 2.07 mm to (125.8, 73.7)
- moved C12 2.07 mm to (125.4, 69.3)
- moved C14 2.07 mm to (122.9, 71.9)
- moved C15 2.07 mm to (122.9, 71.0)
- moved C16 2.07 mm to (113.8, 70.6)
- moved C17 2.07 mm to (111.0, 70.6)
- moved C58 2.07 mm to (118.9, 66.5)
- moved C61 2.07 mm to (117.5, 66.5)
- moved C8 2.07 mm to (111.0, 72.8)
- moved C86 2.07 mm to (117.4, 76.8)
- moved C9 2.07 mm to (122.6, 74.1)
- moved L4 2.07 mm to (112.8, 75.3)
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Routing:
- net Net-(D12-K): track 3.34 -> 110.9 mm, vias 0 -> 1
- net VCC: track 12.7 -> 101.8 mm, vias 2 -> 6
- net +3.3V: track 1.33 -> 37.2 mm
- net /MCU/PICTURE: track 0.00 -> 9.47 mm
- net /MCU/SCL: track 0.00 -> 9.04 mm
- net /MCU/SDA: track 0.00 -> 7.01 mm
- net /MCU/VDD_ARM: track 8.57 -> 13.9 mm
- net +3V3: track 9.37 -> 11.4 mm
- net /Cam/MCSI_D1P: track 36.3 -> 37.0 mm
- net /Cam/MCSI_D1N: track 36.9 -> 37.6 mm
- added copper zone on B.Cu, net +3.3V

Commit message: feat(Hw):Update_Route
Parts:
- SW8: moved to F.Cu
- moved Y2 0.38 mm to (106.3, 88.5)
- moved R17 0.38 mm to (108.5, 90.7)
- moved R18 0.38 mm to (106.7, 90.7)
- moved C3 0.38 mm to (109.0, 88.8)
- moved C4 0.38 mm to (105.7, 86.1)
- turned C21 to 180 degrees
- turned SW8 to 0 degrees
Routing:
- net VBUS: track 37.9 -> 219.5 mm
- net /MCU/UP: track 4.98 -> 131.7 mm, vias 0 -> 2
- net /MCU/DIN_IR: track 0.00 -> 126.3 mm, vias 0 -> 1
- net /MCU/Battery: track 28.8 -> 155.1 mm, vias 0 -> 2
- net +3.3V: track 37.2 -> 156.6 mm, vias 0 -> 1
- net /MCU/RIGHT: track 5.02 -> 122.7 mm, vias 0 -> 2
- net /MCU/LEFT: track 4.98 -> 113.7 mm, vias 0 -> 2
- net /MCU/DOWN: track 4.91 -> 109.0 mm, vias 0 -> 2
- net /MCU/Enable: track 2.53 -> 94.6 mm, vias 0 -> 2
- net /MCU/SDA: track 7.01 -> 72.4 mm, vias 0 -> 3
- net /Buck_Converter/VCC_DDR: track 6.15 -> 70.9 mm, vias 0 -> 2
- net /MCU/PICTURE: track 9.47 -> 72.9 mm, vias 0 -> 2
- net /MCU/SCL: track 9.04 -> 68.5 mm, vias 0 -> 3
- net +1V8: track 3.49 -> 28.0 mm, vias 0 -> 2
- net +3V3: track 11.4 -> 33.1 mm, vias 0 -> 2
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Other:
- outline, holes or cut-outs redrawn

Commit message: feat(Hw):Update_Route_Init_Rear_Board
Parts:
- moved C26 0.45 mm to (111.8, 92.5)
Routing:
- net +3V3: track 33.1 -> 267.4 mm, vias 2 -> 13
- net +1V8: track 28.0 -> 120.1 mm, vias 2 -> 10
- net /MCU/VDD_ARM: track 34.5 -> 98.0 mm, vias 1 -> 4
- net GND: track 15.9 -> 29.5 mm, vias 1 -> 50
- net Net-(F1-Pad1): track 3.18 -> 10.3 mm
- net /MCU/D-: track 34.2 -> 38.0 mm
- net /MCU/D+: track 33.6 -> 37.1 mm
- net Net-(P4-VCONN): track 0.00 -> 3.00 mm
- added copper zone on B.Cu, net GND
- added copper zone on F.Cu, net GND

Commit message: feat(Hw):Update_Schematic_And_Route
Parts:
- moved R25 15.3 mm to (124.9, 128.9)
- moved SW3 15.0 mm to (130.1, 127.3)
- moved C5 14.9 mm to (124.9, 129.9)
- moved R26 14.6 mm to (124.9, 128.0)
- moved C4 14.2 mm to (104.7, 100.4)
- moved Y2 14.2 mm to (105.3, 102.7)
- moved R18 14.2 mm to (106.6, 104.9)
- moved C3 12.9 mm to (107.9, 101.7)
- moved R17 12.8 mm to (107.9, 103.5), turned to -90 degrees
- moved C27 12.6 mm to (104.6, 105.1), turned to 180 degrees
- moved C64 12.5 mm to (117.0, 104.0)
- moved C65 12.5 mm to (117.0, 103.1)
- moved FB2 12.5 mm to (117.3, 105.2)
- moved C39 12.0 mm to (113.4, 104.5)
- moved R29 11.8 mm to (118.3, 107.4)
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Connections:
- J1 pad 1: GND -> +3V3
- J1 pad 10: /Cam/MCSI_D1P -> /Cam/MCSI_D1N
- J1 pad 11: /Cam/MCSI_D1N -> /Cam/MCSI_D1P
- J1 pad 13: /Cam/CSI_SCK -> /Cam/MCSI_CKN
- J1 pad 14: /Cam/CSI_SDA -> /Cam/MCSI_CKP
- J1 pad 16: /Cam/MCSI_RST -> /Cam/MCSI_D0N
- J1 pad 17: GND -> /Cam/MCSI_D0P
- J1 pad 19: +3V3 -> /Cam/MCSI_MCLK
- J1 pad 2: /Cam/MCSI_MCLK -> +3V3
- J1 pad 20: +3V3 -> GND
- J1 pad 4: /Cam/MCSI_D0P -> GND
- J1 pad 5: /Cam/MCSI_D0N -> /Cam/MCSI_RST
- J1 pad 7: /Cam/MCSI_CKP -> /Cam/CSI_SDA
- J1 pad 8: /Cam/MCSI_CKN -> /Cam/CSI_SCK
Routing:
- net /MCU/DOWN: track 109.0 -> 20.6 mm, vias 2 -> 1
- net /MCU/RIGHT: track 122.7 -> 43.1 mm, vias 2 -> 1
- net /MCU/UP: track 131.7 -> 53.1 mm, vias 2 -> 1
- net /MCU/LEFT: track 113.7 -> 38.3 mm, vias 2 -> 1
- net +3V3: track 267.4 -> 209.4 mm, vias 13 -> 9
- net /Cam/CSI_SDA: track 47.6 -> 7.75 mm
- net /Cam/CSI_SCK: track 45.2 -> 7.58 mm
- net /Cam/MCSI_RST: track 43.8 -> 11.5 mm, vias 2 -> 0
- net /Cam/MCSI_MCLK: track 37.1 -> 15.0 mm
- net +1V8: track 120.1 -> 103.5 mm, vias 10 -> 9
- net /MCU/SCL: track 68.2 -> 80.3 mm
- net /MCU/SDA: track 72.0 -> 83.6 mm
- net /MCU/PICTURE: track 72.9 -> 84.4 mm
- net /MCU/DEBUG_RX: track 46.4 -> 57.6 mm
- net /MCU/RECOVERY: track 16.8 -> 25.8 mm
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