File: hardware/Badge-HackGDL-2026.kicad_pcb (KiCad board)
At the start: 2 copper layers, 150 x 100 mm, 131 parts, among them J1 Conn_01x20, J10 Battery, J2 Conn_01x04_Pin, J9 Add_On, P4 USB_C_Plug_USB2.0, Q1 DMG3415U-7, SW1 ON, SW2 SW_Push, SW3 SW_Push, U2 TP4056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

Commit message: feat(Hw):Update_Schematic_And_Route
Parts:
- moved C21 2.39 mm to (200.6, 47.9), turned to 90 degrees
- moved SW3 0.39 mm to (130.1, 126.9)
- moved C5 0.21 mm to (125.0, 129.7)
- moved R25 0.21 mm to (124.9, 128.7)
- moved R26 0.21 mm to (124.9, 127.8)
Connections:
- J1 pad 1: +3V3 -> +3.3V
- J1 pad 2: +3V3 -> +3.3V
Routing:
- net /MCU/DOWN: track 20.6 -> 120.3 mm, vias 1 -> 2
- net /MCU/RIGHT: track 43.1 -> 134.2 mm, vias 1 -> 2
- net /MCU/UP: track 53.1 -> 143.5 mm, vias 1 -> 2
- net /MCU/LEFT: track 38.3 -> 125.0 mm, vias 1 -> 2
- net +3.3V: track 156.6 -> 239.2 mm, vias 1 -> 2
- net +3V3: track 209.4 -> 283.4 mm
- net /Cam/CSI_SDA: track 7.75 -> 53.7 mm, vias 0 -> 2
- net /Cam/CSI_SCK: track 7.58 -> 52.0 mm, vias 0 -> 2
- net /Cam/MCSI_RST: track 11.5 -> 43.1 mm, vias 0 -> 2
- net /Cam/MCSI_MCLK: track 15.0 -> 45.6 mm
- net +1V8: track 103.5 -> 128.0 mm, vias 9 -> 10
- net /MCU/VDD_ARM: track 95.7 -> 108.9 mm
- net /MCU/DIN_IR: track 126.3 -> 138.1 mm
- net /MCU/Enable: track 94.6 -> 106.4 mm
- net /Buck_Converter/VCC_DDR: track 71.0 -> 82.7 mm
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
Commit message: feat(Hw):Update_Route
Routing:
- net GND: vias 39 -> 51
Changed lines of the file:
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@@
 	)
 	(via
+		(at 125.63 118.45)
+		(size 0.6)
+		(drill 0.3)
+		(layers "F.Cu" "B.Cu")
+		(free yes)
+		(net 2)
+	)
+	(via
+		(at 128.76 118.45)
+		(size 0.6)
+		(drill 0.3)
+		(layers "F.Cu" "B.Cu")
+		(free yes)
+		(net 2)
+	)
+	(via
 		(at 95.995 117.165)
 		(size 0.6)
@@
 	)
 	(via
+		(at 146.38 115.7)
+		(size 0.6)
+		(drill 0.3)
+		(layers "F.Cu" "B.Cu")
+		(free yes)
+		(net 2)
+	)
+	(via
 		(at 109.78 112.61)
 		(size 0.6)
@@
 	)
 	(via
+		(at 138 115.92)
+		(size 0.6)
+		(drill 0.3)
+		(layers "F.Cu" "B.Cu")
+		(free yes)
+		(net 2)
+	)
+	(via
 		(at 86.87 128.72)
 		(size 0.6)
@@
 	)
 	(via
+		(at 132.81 115.93)
+		(size 0.6)
+		(drill 0.3)
+		(layers "F.Cu" "B.Cu")
+		(free yes)
+		(net 2)
+	)
+	(via
 		(at 101.015 110.065)
 		(size 0.6)
@@
 	)
 	(via
+		(at 130.69 118.46)
+		(size 0.6)
+		(drill 0.3)
+		(layers "F.Cu" "B.Cu")
+		(free yes)
+		(net 2)
+	)
+	(via
 		(at 119.04 115.37)
 		(size 0.6)
@@
 	)
 	(via
+		(at 127.19 118.45)
+		(size 0.6)
+		(drill 0.3)
+		(layers "F.Cu" "B.Cu")
+		(free yes)
+		(net 2)
+	)
+	(via
 		(at 84.87 130.72)
 		(size 0.6)
@@
 	)
 	(via
+		(at 139.36 115.92)
+		(size 0.6)
+		(drill 0.3)
+		(layers "F.Cu" "B.Cu")
+		(free yes)
+		(net 2)
+	)
+	(via
 		(at 121.97 123.09)
 		(size 0.6)
@@
 	)
 	(via
+		(at 147.9 118.47)
+		(size 0.6)
+		(drill 0.3)
+		(layers "F.Cu" "B.Cu")
+		(free yes)
+		(net 2)
+	)
+	(via
 		(at 85.87 130.72)
 		(size 0.6)
@@
 	)
 	(via
+		(at 131.72 115.95)
+		(size 0.6)
+		(drill 0.3)
+		(layers "F.Cu" "B.Cu")
+		(free yes)
+		(net 2)
+	)
+	(via
 		(at 93.035 115.155)
 		(size 0.6)
@@
 	)
 	(via
+		(at 142.03 118.45)
+		(size 0.6)
+		(drill 0.3)
+		(layers "F.Cu" "B.Cu")
+		(free yes)
+		(net 2)
+	)
+	(via
 		(at 109 65)
 		(size 0.6)
@@
 		(net 2)
 	)
+	(via
+		(at 146.4 118.45)
+		(size 0.6)
+		(drill 0.3)
+		(layers "F.Cu" "B.Cu")
+		(free yes)
+		(net 2)
+	)
 	(segment
 		(start 116.25 72.95)
@@
 	)
 	(segment
-		(start 99.51 130.91)
-		(end 98.16 129.56)
+		(start 98.16 129.56)
+		(end 98.16 127.17)
 		(width 0.5)
 		(layer "B.Cu")
@@
 	)
 	(segment
-		(start 162.46 69.84)
-		(end 162.46 127.99)
-		(width 0.5)
-		(layer "B.Cu")
-		(net 31)
-	)
-	(segment
 		(start 83.665 125.165)
 		(end 84.94 126.44)
@@
 	)
 	(segment
-		(start 162.47 128)
-		(end 162.47 128.96)
-		(width 0.5)
-		(layer "B.Cu")
-		(net 31)
-	)
-	(segment
 		(start 163.2 69.16)
 		(end 162.52 69.84)
@@
 	)
 	(segment
+		(start 160.52 130.91)
+		(end 99.51 130.91)
+		(width 0.5)
+		(layer "B.Cu")
+		(net 31)
+	)
+	(segment
 		(start 169.51512 57.32012)
 		(end 169.525 57.33)
@@
 	)
 	(segment
+		(start 162.46 69.84)
+		(end 162.46 128.97)
+		(width 0.5)
+		(layer "B.Cu")
+		(net 31)
+	)
+	(segment
 		(start 98.83 126.5)
 		(end 98.83 126.44)
@@
 	)
 	(segment
-		(start 98.16 129.56)
-		(end 98.16 127.17)
+		(start 99.51 130.91)
+		(end 98.16 129.56)
 		(width 0.5)
 		(layer "B.Cu")
@@
 	)
 	(segment
-		(start 162.47 128.96)
-		(end 160.52 130.91)
-		(width 0.5)
-		(layer "B.Cu")
-		(net 31)
-	)
-	(segment
 		(start 162.46 68.38)
 		(end 162.46 69.16)
@@
 	)
 	(segment
-		(start 162.46 127.99)
-		(end 162.47 128)
+		(start 162.46 128.97)
+		(end 160.52 130.91)
 		(width 0.5)
 		(layer "B.Cu")
@@
 		(width 0.5)
 		(layer "B.Cu")
-		(net 31)
-	)
-	(segment
-		(start 160.52 130.91)
-		(end 99.51 130.91)
-		(width 0.5)
-		(layer "B.Cu")

Commit message: feat(Hw):Update_Shematic_And_PCB
Parts:
- added J4: Conn_01x08, Connector_PinSocket_2.54mm:PinSocket_1x08_P2.54mm_Vertical, B.Cu at (164.3, 42.2)
- added J5: Conn_01x08, Connector_PinSocket_2.54mm:PinSocket_1x08_P2.54mm_Vertical, B.Cu at (217.4, 102.7)
- added J6: Conn_01x08, Connector_PinSocket_2.54mm:PinSocket_1x08_P2.54mm_Vertical, B.Cu at (154.5, 128.2)
- added J7: Conn_01x08, Connector_PinSocket_2.54mm:PinSocket_1x08_P2.54mm_Vertical, B.Cu at (75.5, 84.3)
- moved J2 5.47 mm to (81.8, 79.6)
Routing:
- net +3.3V: track 239.2 -> 233.0 mm
- net +3V3: track 283.4 -> 277.8 mm
- net /MCU/DEBUG_TX: track 54.5 -> 49.1 mm
- net /MCU/DEBUG_RX: track 57.6 -> 52.2 mm
- net VBUS: track 217.7 -> 215.6 mm
- net /MCU/Battery: track 158.1 -> 157.4 mm
Other:
- outline, holes or cut-outs redrawn
