File: hardware/Buck_Converter.kicad_sch (KiCad schematic)
At the start: 40 parts, among them U7 EA3059

Commit message: feat(Hw):Update_Schematic
Parts:
- removed D3, D4, D5, D6: LED, LED_SMD:LED_0603_1608Metric, symbol Device:LED
- removed R39: 330, Resistor_SMD:R_0402_1005Metric, symbol Device:R_Small
- removed R41, R42, R43: 50, Resistor_SMD:R_0603_1608Metric, symbol Device:R_Small

Commit message: feat(Hw):Update_3Dmodels_And_Rear_Board
Other:
- company: (none) -> Electronic Cats
- title: (none) -> Badge-HackGDL-2026
Changed lines of the file:
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@@
 	(generator_version "9.0")
 	(paper "A4")
+	(title_block
+		(title "Badge-HackGDL-2026")
+		(date "2026-01-15")
+		(rev "v1.0")
+		(company "Electronic Cats")
+		(comment 1 "Lizeth Gallegos Martínez")
+	)
 	(text "Fixed LXn Switching \nFrequency: 1.5MHz"
 		(exclude_from_sim no)
