File: hardware/Otros.kicad_sch (KiCad schematic)
At the start: 11 parts, among them J9 Add_On

Commit message: feat(Hw):Update_Schematic_And_Floorplan
Other:
- moved on the sheet: J9
Changed lines of the file:
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@@
 	)
 	(junction
-		(at 33.02 43.18)
+		(at 42.672 46.99)
 		(diameter 0)
 		(color 0 0 0 0)
@@
 	)
 	(no_connect
-		(at 36.068 48.26)
+		(at 45.72 52.07)
 	)
 	(no_connect
-		(at 48.768 48.26)
+		(at 58.42 52.07)
 	)
 	(polyline
@@
 	(wire
 		(pts
-			(xy 29.21 43.18) (xy 33.02 43.18)
+			(xy 38.862 46.99) (xy 42.672 46.99)
 		)
 		(stroke
@@
 	(wire
 		(pts
-			(xy 56.388 44.45) (xy 56.388 43.18)
+			(xy 66.04 48.26) (xy 66.04 46.99)
 		)
 		(stroke
@@
 	(wire
 		(pts
-			(xy 35.56 45.72) (xy 36.068 45.72)
+			(xy 45.212 49.53) (xy 45.72 49.53)
 		)
 		(stroke
@@
 	(wire
 		(pts
-			(xy 48.768 45.72) (xy 49.53 45.72)
+			(xy 58.42 49.53) (xy 59.182 49.53)
 		)
 		(stroke
@@
 	(wire
 		(pts
-			(xy 56.388 43.18) (xy 48.768 43.18)
+			(xy 66.04 46.99) (xy 58.42 46.99)
 		)
 		(stroke
@@
 	(wire
 		(pts
-			(xy 33.02 39.37) (xy 33.02 43.18)
-		)
-		(stroke
-			(width 0)
-			(type default)
-		)
-	)
-	(wire
-		(pts
-			(xy 33.02 43.18) (xy 36.068 43.18)
+			(xy 42.672 43.18) (xy 42.672 46.99)
+		)
+		(stroke
+			(width 0)
+			(type default)
+		)
+	)
+	(wire
+		(pts
+			(xy 42.672 46.99) (xy 45.72 46.99)
 		)
 		(stroke
@@
 		)
 	)
-	(label "UP"
+	(hierarchical_label "UP"
+		(shape input)
 		(at 153.67 82.55 180)
 		(effects
@@
 				(size 1.27 1.27)
 			)
-			(justify right bottom)
-		)
-	)
-	(label "DOWN"
+			(justify right)
+		)
+	)
+	(hierarchical_label "PICTURE"
+		(shape input)
+		(at 43.18 102.87 180)
+		(effects
+			(font
+				(size 1.27 1.27)
+			)
+			(justify right)
+		)
+	)
+	(hierarchical_label "SDA"
+		(shape bidirectional)
+		(at 45.212 49.53 180)
+		(effects
+			(font
+				(size 1.27 1.27)
+			)
+			(justify right)
+		)
+	)
+	(hierarchical_label "DOWN"
+		(shape input)
 		(at 154.94 63.5 180)
 		(effects
@@
 				(size 1.27 1.27)
 			)
-			(justify right bottom)
-		)
-	)
-	(label "LEFT"
-		(at 154.94 26.67 180)
+			(justify right)
+		)
+	)
+	(hierarchical_label "SCL"
+		(shape bidirectional)
+		(at 59.182 49.53 0)
 		(effects
 			(font
 				(size 1.27 1.27)
 			)
-			(justify right bottom)
-		)
-	)
-	(label "PICTURE"
-		(at 43.18 102.87 180)
+			(justify left)
+		)
+	)
+	(hierarchical_label "+3.3v"
+		(shape input)
+		(at 38.862 46.99 180)
 		(effects
 			(font
 				(size 1.27 1.27)
 			)
-			(justify right bottom)
-		)
-	)
-	(label "RIGHT"
+			(justify right)
+		)
+	)
+	(hierarchical_label "RIGHT"
+		(shape input)
 		(at 154.94 46.99 180)
 		(effects
@@
 				(size 1.27 1.27)
 			)
-			(justify right bottom)
-		)
-	)
-	(hierarchical_label "SDA"
-		(shape bidirectional)
-		(at 35.56 45.72 180)
-		(effects
-			(font
-				(size 1.27 1.27)
-			)
 			(justify right)
 		)
 	)
-	(hierarchical_label "SCL"
-		(shape bidirectional)
-		(at 49.53 45.72 0)
-		(effects
-			(font
-				(size 1.27 1.27)
-			)
-			(justify left)
-		)
-	)
-	(hierarchical_label "+3.3v"
+	(hierarchical_label "LEFT"
 		(shape input)
-		(at 29.21 43.18 180)
+		(at 154.94 26.67 180)
 		(effects
 			(font
@@
 	(symbol
 		(lib_id "Connector_Generic:Conn_02x03_Odd_Even")
-		(at 41.148 45.72 0)
+		(at 50.8 49.53 0)
 		(unit 1)
 		(exclude_from_sim no)
@@
 		(fields_autoplaced yes)
 		(property "Reference" "J9"
-			(at 42.418 36.83 0)
+			(at 52.07 40.64 0)
 			(effects
 				(font
@@
 		)
 		(property "Value" "Add_On"
-			(at 42.418 39.37 0)
+			(at 52.07 43.18 0)
 			(effects
 				(font
@@
 		)
 		(property "Footprint" "Connector_PinSocket_2.54mm:PinSocket_2x03_P2.54mm_Vertical"
-			(at 41.148 45.72 0)
+			(at 50.8 49.53 0)
 			(effects
 				(font
@@
 		)
 		(property "Datasheet" "~"
-			(at 41.148 45.72 0)
+			(at 50.8 49.53 0)
 			(effects
 				(font
@@
 		)
 		(property "Description" "Generic connector, double row, 02x03, odd/even pin numbering scheme (row 1 odd numbers, row 2 even numbers), script generated (kicad-library-utils/schlib/autogen/connector/)"
-			(at 41.148 45.72 0)
+			(at 50.8 49.53 0)
 			(effects
 				(font
@@
 		)
 		(property "LCSC#" "C5116527"
-			(at 41.148 45.72 0)
+			(at 50.8 49.53 0)
 			(effects
 				(font
@@
 		)
 		(property "Proveedor" "JLCPCB"
-			(at 41.148 45.72 0)
+			(at 50.8 49.53 0)
 			(effects
 				(font
@@
 		)
 		(property "Height" ""
-			(at 41.148 45.72 0)
+			(at 50.8 49.53 0)
 			(effects
 				(font
@@
 		)
 		(property "Manufacturer_Name" ""
-			(at 41.148 45.72 0)
+			(at 50.8 49.53 0)
 			(effects
 				(font
@@
 		)
 		(property "Mouser Part Number" ""
-			(at 41.148 45.72 0)
+			(at 50.8 49.53 0)
 			(effects
 				(font
@@
 		)
 		(property "Mouser Price/Stock" ""
-			(at 41.148 45.72 0)
+			(at 50.8 49.53 0)
 			(effects
 				(font
@@
 		)
 		(property "Availability" ""
-			(at 41.148 45.72 0)
+			(at 50.8 49.53 0)
 			(effects
 				(font
@@
 		)
 		(property "Check_prices" ""
-			(at 41.148 45.72 0)
+			(at 50.8 49.53 0)
 			(effects
 				(font
@@
 		)
 		(property "Description_1" ""
-			(at 41.148 45.72 0)
+			(at 50.8 49.53 0)
 			(effects
 				(font
@@
 		)
 		(property "MANUFACTURER" ""
-			(at 41.148 45.72 0)
+			(at 50.8 49.53 0)
 			(effects
 				(font
@@
 		)
 		(property "MAXIMUM_PACKAGE_HEIGHT" ""
-			(at 41.148 45.72 0)
+			(at 50.8 49.53 0)
 			(effects
 				(font
@@
 		)
 		(property "MF" ""
-			(at 41.148 45.72 0)
+			(at 50.8 49.53 0)
 			(effects
 				(font
@@
 		)
 		(property "MP" ""
-			(at 41.148 45.72 0)
+			(at 50.8 49.53 0)
 			(effects
 				(font
@@
 		)
 		(property "PARTREV" ""
-			(at 41.148 45.72 0)
+			(at 50.8 49.53 0)
 			(effects
 				(font
@@
 		)
 		(property "Package" ""
-			(at 41.148 45.72 0)
+			(at 50.8 49.53 0)
 			(effects
 				(font
@@
 		)
 		(property "Price" ""
-			(at 41.148 45.72 0)
+			(at 50.8 49.53 0)
 			(effects
 				(font
@@
 		)
 		(property "STANDARD" ""
-			(at 41.148 45.72 0)
+			(at 50.8 49.53 0)
 			(effects
 				(font
@@
 		)
 		(property "SnapEDA_Link" ""
-			(at 41.148 45.72 0)
+			(at 50.8 49.53 0)
 			(effects
 				(font
@@
 		)
 		(property "JLCPCB" ""
-			(at 41.148 45.72 0)
+			(at 50.8 49.53 0)
 			(effects
 				(font
@@
 		)
 		(property "Manufacter Number" ""
-			(at 41.148 45.72 0)
+			(at 50.8 49.53 0)
 			(effects
 				(font
@@
 		)
 		(property "Mnfr#" ""
-			(at 41.148 45.72 0)
+			(at 50.8 49.53 0)
 			(effects
 				(font
@@
 		)
 		(property "SNAPEDA_PN" ""
-			(at 41.148 45.72 0)
+			(at 50.8 49.53 0)
 			(effects
 				(font
@@
 	(symbol
 		(lib_id "power:+3.3V")
-		(at 33.02 39.37 0)
+		(at 42.672 43.18 0)
 		(unit 1)
 		(exclude_from_sim no)
@@
 		(fields_autoplaced yes)
 		(property "Reference" "#PWR089"
-			(at 33.02 43.18 0)
+			(at 42.672 46.99 0)
 			(effects
 				(font
@@
 		)
 		(property "Value" "+3.3V"
-			(at 33.02 34.29 0)
+			(at 42.672 38.1 0)
 			(effects
 				(font
@@
 		)
 		(property "Footprint" ""
-			(at 33.02 39.37 0)
+			(at 42.672 43.18 0)
 			(effects
 				(font
@@
 		)
 		(property "Datasheet" ""
-			(at 33.02 39.37 0)
+			(at 42.672 43.18 0)
 			(effects
 				(font
@@
 		)
 		(property "Description" "Power symbol creates a global label with name \"+3.3V\""
-			(at 33.02 39.37 0)
+			(at 42.672 43.18 0)
 			(effects
 				(font
@@
 	(symbol
 		(lib_id "power:GND")
-		(at 56.388 44.45 0)
+		(at 66.04 48.26 0)
 		(unit 1)
 		(exclude_from_sim no)
@@
 		(dnp no)
 		(property "Reference" "#PWR0153"
-			(at 56.388 50.8 0)
+			(at 66.04 54.61 0)
 			(effects
 				(font
@@
 		)
 		(property "Value" "GND"
-			(at 56.388 48.006 0)
+			(at 66.04 51.816 0)
 			(effects
 				(font
@@
 		)
 		(property "Footprint" ""
-			(at 56.388 44.45 0)
+			(at 66.04 48.26 0)
 			(effects
 				(font
@@
 		)
 		(property "Datasheet" ""
-			(at 56.388 44.45 0)
+			(at 66.04 48.26 0)
 			(effects
 				(font
@@
 		)
 		(property "Description" "Power symbol creates a global label with name \"GND\" , ground"
-			(at 56.388 44.45 0)
-			(effects
-				(font
+			(at 66.04 48.26 0)
+			(effects
+				(font

Commit message: feat(Hw):Update_Schematic_And_BOM
Parts:
- added R10, R4: 4.7K, Capacitor_SMD:C_0603_1608Metric, symbol Device:R
Connections:
- net +3.3V: now also R10.1, R4.1
- net SCL: now also R4.2
- net SDA: now also R10.2

Commit message: feat(Hw):Update_Schematic_And_Floorplan
Parts:
- SW8: footprint Button_Switch_SMD:SW_SPST_TL3342 -> Footprints:Button_6.6x6.5; LCSC# C318889 -> C480263; manf# TL3342F160QG -> (none)
Changed lines of the file:
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@@
 			)
 		)
-		(property "Footprint" "Button_Switch_SMD:SW_SPST_TL3342"
+		(property "Footprint" "Footprints:Button_6.6x6.5"
 			(at 50.8 97.79 0)
 			(effects
@@
 			)
 		)
-		(property "manf#" "TL3342F160QG"
+		(property "manf#" ""
 			(at 50.8 102.87 0)
 			(effects
@@
 			)
 		)
-		(property "LCSC#" "C318889"
+		(property "LCSC#" "C480263"
 			(at 50.8 102.87 0)
 			(effects

Commit message: feat(Hw):Update_Floorplan_And_Route
Parts:
- added C21: 100nF, Capacitor_SMD:C_0402_1005Metric, symbol Device:C_Small
- added D7: WS2812E-1313, Footprints:WS2812E-1313, symbol LED:WS2812B
- added R28: 470R, Resistor_SMD:R_0603_1608Metric, symbol Device:R_Small
Connections:
- net +3.3V: now also C21.1, D7.1 (VDD)
- net GND: now also C21.2, D7.3 (VSS)
- new net: D7.4 (DIN), R28.2
- new net DIN_IR: R28.1
- no-connect marks 2 -> 3
Other:
- note added: "BUTTONS"
- note added: "NEOPIXEL"
- moved on the sheet: C19, C2, C33, C37, C43, J9, R10, R4, SW4, SW5, SW6, SW7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

Commit message: feat(Hw):Update_3Dmodels_And_Rear_Board
Other:
- company: (none) -> Electronic Cats
- title: (none) -> Badge-HackGDL-2026
Changed lines of the file:
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@@
 	(generator_version "9.0")
 	(paper "A5")
+	(title_block
+		(title "Badge-HackGDL-2026")
+		(date "2026-01-15")
+		(rev "v1.0")
+		(company "Electronic Cats")
+		(comment 1 "Lizeth Gallegos Martínez")
+	)
 	(text "BUTTONS\n"
 		(exclude_from_sim no)
