File: hardware/Support pins.kicad_sch (KiCad schematic)
At the start: 4 parts, among them J4 Conn_01x08, J5 Conn_01x08, J6 Conn_01x08, J7 Conn_01x08

Commit message: feat(Hw):Update_BOM
Parts:
- J4, J5, J6, J7: LCSC# (none) -> C5224027
Changed lines of the file:
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@@
+			)
+		)
+		(property "LCSC#" "C5224027"
+			(at 135.89 57.15 0)
+			(effects
+				(font
+					(size 1.27 1.27)
+				)
+				(hide yes)
 			)
 		)
@@
 			)
 		)
+		(property "LCSC#" "C5224027"
+			(at 91.44 57.15 0)
+			(effects
+				(font
+					(size 1.27 1.27)
+				)
+				(hide yes)
+			)
+		)
 		(pin "6"
 		)
@@
 			)
 		)
+		(property "LCSC#" "C5224027"
+			(at 113.03 57.15 0)
+			(effects
+				(font
+					(size 1.27 1.27)
+				)
+				(hide yes)
+			)
+		)
 		(pin "6"
 		)
@@
 			(at 68.58 57.15 0)
 			(effects
+				(font
+					(size 1.27 1.27)
+				)
+				(hide yes)
+			)
+		)
+		(property "LCSC#" "C5224027"
+			(at 68.58 57.15 0)
+			(effects
