File: hardware/Cam.kicad_sch (KiCad schematic)
At the start: 3 parts, among them J1 Conn_01x20, J3 FLEX_TO_CAM

Commit message: feat(Hw):Update_BOM
Parts:
- J1: LCSC# (none) -> C2906119
Changed lines of the file:
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@@
+			)
+		)
+		(property "LCSC#" "C2906119"
+			(at 157.48 62.23 0)
+			(effects
+				(font
+					(size 1.27 1.27)
+				)
+				(hide yes)
 			)
 		)

Commit message: feat(Hw):Update_BOM
Parts:
- removed J3: FLEX_TO_CAM, symbol Connector:Conn_01x01_Pin
- FID1: manf# https://www.luckfox.com/EN-SC3336-3MP-Camera-B -> (none)
Connections:
- no-connect marks 1 -> 0
Changed lines of the file:
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@@
 		(color 0 0 0 0)
-	)
-	(no_connect
-		(at 58.42 67.31)
 	)
 	(wire
@@
 				(path "/aee06ce3-1da5-4230-bf8f-9d1068f7ddd5/81efd129-08c1-4996-9ee0-a58d47ad59bf"
 					(reference "J1")
-					(unit 1)
-				)
-			)
-		)
-	)
-	(symbol
-		(lib_id "Connector:Conn_01x01_Pin")
-		(at 53.34 67.31 0)
-		(unit 1)
-		(exclude_from_sim no)
-		(in_bom yes)
-		(on_board yes)
-		(dnp no)
-		(fields_autoplaced yes)
-		(property "Reference" "J3"
-			(at 53.975 62.23 0)
-			(effects
-				(font
-					(size 1.27 1.27)
-				)
-			)
-		)
-		(property "Value" "FLEX_TO_CAM"
-			(at 53.975 64.77 0)
-			(effects
-				(font
-					(size 1.27 1.27)
-				)
-			)
-		)
-		(property "Footprint" ""
-			(at 53.34 67.31 0)
-			(effects
-				(font
-					(size 1.27 1.27)
-				)
-				(hide yes)
-			)
-		)
-		(property "Datasheet" "~"
-			(at 53.34 67.31 0)
-			(effects
-				(font
-					(size 1.27 1.27)
-				)
-				(hide yes)
-			)
-		)
-		(property "Description" "Generic connector, single row, 01x01, script generated"
-			(at 53.34 67.31 0)
-			(effects
-				(font
-					(size 1.27 1.27)
-				)
-				(hide yes)
-			)
-		)
-		(property "LCSC#" "C22434842"
-			(at 53.34 67.31 0)
-			(effects
-				(font
-					(size 1.27 1.27)
-				)
-				(hide yes)
-			)
-		)
-		(pin "1"
-		)
-		(instances
-			(project "Cam"
-				(path "/4f679915-e6d1-4835-bbdc-b9d0e7615f17"
-					(reference "J?")
-					(unit 1)
-				)
-			)
-			(project "Badge-HackGDL-2026"
-				(path "/aee06ce3-1da5-4230-bf8f-9d1068f7ddd5/81efd129-08c1-4996-9ee0-a58d47ad59bf"
-					(reference "J3")
 					(unit 1)
 				)
@@
 			)
 		)
-		(property "manf#" "https://www.luckfox.com/EN-SC3336-3MP-Camera-B"
+		(property "manf#" ""
 			(at 53.34 54.61 0)
 			(effects
