File: hardware/Rear-Badge-HackGDL-2026/Rear-Badge-HackGDL-2026.kicad_pcb (KiCad board)
At the start: 2 copper layers, 150 x 100 mm, 0 parts

Commit message: feat(Hw):Update_Shematic_And_PCB
Parts:
- added J4: Conn_01x08, Connector_PinHeader_2.54mm:PinHeader_1x08_P2.54mm_Vertical, F.Cu at (166.7, 51.3)
- added J5: Conn_01x08, Connector_PinHeader_2.54mm:PinHeader_1x08_P2.54mm_Vertical, F.Cu at (219.7, 111.7)
- added J6: Conn_01x08, Connector_PinHeader_2.54mm:PinHeader_1x08_P2.54mm_Vertical, F.Cu at (156.9, 137.2)
- added J7: Conn_01x08, Connector_PinHeader_2.54mm:PinHeader_1x08_P2.54mm_Vertical, F.Cu at (77.8, 93.4)
Other:
- outline, holes or cut-outs redrawn
