File: Add-ons/Add-on-Pescadito-HackGDL/Orange_Fish.kicad_sch (KiCad schematic)
At the start: 16 parts, among them J6 Conn_02x03_Odd_Even, SW11 SW_RST, SW12 On, U6 PY32F002AA15M6TU

Commit message: feat(Hw):Update_Labels
Parts:
- D26: value Red -> White; LCSC# C965812 -> C84258
- D27, D28, D29, D30: value Red -> Orange; LCSC# C965812 -> C434437
Changed lines of the file:
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@@
 			)
 		)
-		(property "Value" "Red"
+		(property "Value" "Orange"
 			(at 184.023 89.154 0)
 			(effects
@@
 			)
 		)
-		(property "LCSC#" "C965812"
+		(property "LCSC#" "C434437"
 			(at 184.15 92.71 0)
 			(effects
@@
 			)
 		)
-		(property "Value" "Red"
+		(property "Value" "Orange"
 			(at 184.2135 58.674 0)
 			(effects
@@
 			)
 		)
-		(property "LCSC#" "C965812"
+		(property "LCSC#" "C434437"
 			(at 184.15 62.23 0)
 			(effects
@@
 			)
 		)
-		(property "Value" "Red"
+		(property "Value" "Orange"
 			(at 184.2135 42.799 0)
 			(effects
@@
 			)
 		)
-		(property "LCSC#" "C965812"
+		(property "LCSC#" "C434437"
 			(at 184.15 46.99 0)
 			(effects
@@
 			)
 		)
-		(property "Value" "Red"
+		(property "Value" "Orange"
 			(at 184.2135 73.914 0)
 			(effects
@@
 			)
 		)
-		(property "LCSC#" "C965812"
+		(property "LCSC#" "C434437"
 			(at 184.15 77.47 0)
 			(effects
@@
 			)
 		)
-		(property "Value" "Red"
+		(property "Value" "White"
 			(at 184.2135 29.464 0)
 			(effects
@@
 			)
 		)
-		(property "LCSC#" "C965812"
+		(property "LCSC#" "C84258"
 			(at 184.15 33.02 0)
 			(effects
